Commit message: add collision and inertial

File: urdf/bot.urdf (robot description, URDF)
Before this commit: robot bot, 4 links, 3 joints
Links:
- link caster: mass None -> 0.2; geometry collision geometry ; visual sphere radius=0.05
- link left_wheel: mass None -> 0.1; geometry collision cylinder length=0.05 radius=0.1; visual cylinder length=0.05 radius=0.1
- link right_wheel: mass None -> 0.1; geometry collision cylinder length=0.05 radius=0.1; visual cylinder length=0.05 radius=0.1
