Commit message: switch to xacro

File: urdf/bot.urdf.xacro (robot description, xacro)
@@ -1,4 +1,8 @@
 <?xml version="1.0"?>
-<robot name="bot">
+<robot xmlns:xacro="http://www.ros.org/wiki/xacro" name="bot">
+    <xacro:property name="PI" value="3.141592653589793" />
+    <xacro:property name="base_width" value="0.4" />
+    <xacro:property name="base_depth" value="0.2" />
+    <xacro:property name="base_height" value="0.1" />
     <!-- define colors -->
     <material name="blue">
@@ -17,5 +21,5 @@
         <visual>
             <geometry>
-                <box size="0.4 0.2 0.1" />
+                <box size="${base_width} ${base_depth} ${base_height}" />
             </geometry>
             <material name="white" />
@@ -23,8 +27,7 @@
         <collision>
             <geometry>
-                <box size="0.4 0.2 0.1" />
+                <box size="${base_width} ${base_depth} ${base_height}" />
             </geometry>
         </collision>
-        >
         <inertial>
             <mass value="1" />
@@ -35,5 +38,5 @@
         <parent link="base_link" />
         <child link="left_wheel" />
-        <origin rpy="1.5707963267948966 0 0" xyz="0.1 0.13 0" />
+        <origin rpy="${PI/2} 0 0" xyz="0.1 0.13 0" />
         <axis rpy="0 0 0" xyz="0 0 1" />
     </joint>
@@ -51,6 +54,6 @@
         </collision>
         <inertial>
-            <mass value="0.1"/>
-           <inertia ixx="0.1" ixy="0.0" ixz="0.0" iyy="0.1" iyz="0.0" izz="0.1"/>
+            <mass value="0.1" />
+            <inertia ixx="0.1" ixy="0.0" ixz="0.0" iyy="0.1" iyz="0.0" izz="0.1" />
         </inertial>
     </link>
@@ -74,6 +77,6 @@
         </collision>
         <inertial>
-            <mass value="0.1"/>
-           <inertia ixx="0.1" ixy="0.0" ixz="0.0" iyy="0.1" iyz="0.0" izz="0.1"/>
+            <mass value="0.1" />
+            <inertia ixx="0.1" ixy="0.0" ixz="0.0" iyy="0.1" iyz="0.0" izz="0.1" />
         </inertial>
     </link>
@@ -93,11 +96,11 @@
             <geometry>
                 <geometry>
-                    <sphere radius="0.05"/>
+                    <sphere radius="0.05" />
                 </geometry>
             </geometry>
         </collision>
         <inertial>
-            <mass value="0.2"/>
-            <inertia ixx="0.1" ixy="0.0" ixz="0.0" iyy="0.1" iyz="0.0" izz="0.1"/>
+            <mass value="0.2" />
+            <inertia ixx="0.1" ixy="0.0" ixz="0.0" iyy="0.1" iyz="0.0" izz="0.1" />
         </inertial>
     </link>

Commit message: update xacro

File: urdf/bot.urdf.xacro (robot description, xacro)
@@ -1,8 +1,19 @@
 <?xml version="1.0"?>
 <robot xmlns:xacro="http://www.ros.org/wiki/xacro" name="bot">
+    <!-- constants -->
     <xacro:property name="PI" value="3.141592653589793" />
     <xacro:property name="base_width" value="0.4" />
     <xacro:property name="base_depth" value="0.2" />
     <xacro:property name="base_height" value="0.1" />
+    <xacro:property name="x_offset" value="0.1" />
+    <xacro:property name="wheel_width" value="0.05" />
+    <xacro:property name="wheel_gap" value="0.005" />
+    <!-- macros -->
+    <xacro:macro name="box_inertial" params="mass x y z">
+        <inertial>
+            <mass value="${mass}" />
+            <inertia ixx="${1/12*mass*(y*y+z*z)}" ixy="0.0" ixz="0.0" iyy="${1/12*mass*(x*x+z*z)}" iyz="0.0" izz="${1/12*mass*(y*y+x*x)}" />
+        </inertial>
+    </xacro:macro>
     <!-- define colors -->
     <material name="blue">
@@ -30,13 +41,10 @@
             </geometry>
         </collision>
-        <inertial>
-            <mass value="1" />
-            <inertia ixx="0.0042" ixy="0.0" ixz="0.0" iyy="0.0142" iyz="0.0" izz="0.0167" />
-        </inertial>
+        <xacro:box_inertial mass="1" x="${base_width}" y="${base_depth}" z="${base_height}"/>
     </link>
     <joint name="base_to_left_wheel" type="continuous">
         <parent link="base_link" />
         <child link="left_wheel" />
-        <origin rpy="${PI/2} 0 0" xyz="0.1 0.13 0" />
+        <origin rpy="${PI/2} 0 0" xyz="${x_offset} ${base_depth/2+wheel_gap+wheel_width/2} 0" />
         <axis rpy="0 0 0" xyz="0 0 1" />
     </joint>
@@ -61,5 +69,6 @@
         <parent link="base_link" />
         <child link="right_wheel" />
-        <origin rpy="1.5707963267948966 0 0" xyz="0.1 -0.13 0" />
+        <origin rpy="${PI/2} 0 0" xyz="${x_offset} ${-(base_depth/2+wheel_gap+wheel_width/2)} 0" />
+        <!-- <origin rpy="1.5707963267948966 0 0" xyz="0.1 -0.13 0" /> -->
         <axis rpy="0 0 0" xyz="0 0 1" />
     </joint>

Commit message: update urdf with diff drive plugin

File: urdf/bot.urdf.xacro (robot description, xacro)
@@ -41,5 +41,23 @@
             </geometry>
         </collision>
-        <xacro:box_inertial mass="1" x="${base_width}" y="${base_depth}" z="${base_height}"/>
+    </link>
+    <gazebo reference="base_link">
+        <material>Gazebo/White</material>
+    </gazebo>
+    <joint name="base_link-base_footprint" type="fixed">
+        <origin rpy="0 0 0" xyz="0 0 -0.15" />
+        <parent link="base_link" />
+        <child link="base_footprint" />
+    </joint>
+    <!-- Base footprint is on the ground under the robot -->
+    <link name="base_footprint" />
+    <joint name="base_link-base_inertial" type="fixed">
+        <origin rpy="0 0 0" xyz="0 0 0" />
+        <parent link="base_link" />
+        <child link="base_inertial" />
+    </joint>
+    <!-- Inertial link stores the robot's inertial information -->
+    <link name="base_inertial">
+        <xacro:box_inertial mass="1" x="${base_width}" y="${base_depth}" z="${base_height}" />
     </link>
     <joint name="base_to_left_wheel" type="continuous">
@@ -66,4 +84,9 @@
         </inertial>
     </link>
+    <gazebo reference="left_wheel">
+        <mu1>1.0</mu1>
+        <mu2>1.0</mu2>
+        <material>Gazebo/Black</material>
+    </gazebo>
     <joint name="base_to_right_wheel" type="continuous">
         <parent link="base_link" />
@@ -90,8 +113,15 @@
         </inertial>
     </link>
-    <joint name="base_to_caster" type="fixed">
+    <gazebo reference="right_wheel">
+        <mu1>1.0</mu1>
+        <mu2>1.0</mu2>
+        <material>Gazebo/Black</material>
+    </gazebo>
+    <joint name="base_to_caster" type="revolute">
         <parent link="base_link" />
         <child link="caster" />
         <origin xyz="-0.15 0 -0.05" />
+        <limit lower="0" upper="0" effort="0" velocity="0" />
+        <axis rpy="0 0 0" xyz="0 0 1" />
     </joint>
     <link name="caster">
@@ -104,7 +134,5 @@
         <collision>
             <geometry>
-                <geometry>
-                    <sphere radius="0.05" />
-                </geometry>
+                <sphere radius="0.05" />
             </geometry>
         </collision>
@@ -114,3 +142,28 @@
         </inertial>
     </link>
+    <gazebo reference="caster">
+        <mu1>0.0</mu1>
+        <mu2>0.0</mu2>
+        <material>Gazebo/Purple</material>
+    </gazebo>
+    <!-- differential_drive_controller plugin -->
+    <gazebo>
+        <plugin name="differential_drive_controller" filename="libgazebo_ros_diff_drive.so">
+            <ros>
+                <!-- Set namespace -->
+                <namespace>/bot</namespace>
+                <!-- <argument>cmd_vel:=cmd_demo</argument>
+                <argument>odom:=odom_demo</argument> -->
+            </ros>
+            <update_rate>100</update_rate>
+            <left_joint>base_to_left_wheel</left_joint>
+            <right_joint>base_to_right_wheel</right_joint>
+            <wheel_separation>0.26</wheel_separation>
+            <wheel_diameter>0.2</wheel_diameter>
+            <odometry_frame>odom</odometry_frame>
+            <max_wheel_torque>20</max_wheel_torque>
+            <!-- Wheel acceleration, in rad/s^2, defaults to 0.0 rad/s^2 -->
+            <max_acceleration>1.0</max_acceleration>
+        </plugin>
+    </gazebo>
 </robot>

Commit message: update urdf with gazebo decors

File: urdf/bot.urdf.xacro (robot description, xacro)
@@ -1,23 +1,7 @@
 <?xml version="1.0"?>
 <robot xmlns:xacro="http://www.ros.org/wiki/xacro" name="bot">
-    <!-- constants -->
-    <xacro:property name="PI" value="3.141592653589793" />
-    <xacro:property name="base_width" value="0.4" />
-    <xacro:property name="base_depth" value="0.2" />
-    <xacro:property name="base_height" value="0.1" />
-    <xacro:property name="x_offset" value="0.1" />
-    <xacro:property name="wheel_width" value="0.05" />
-    <xacro:property name="wheel_gap" value="0.005" />
-    <!-- macros -->
-    <xacro:macro name="box_inertial" params="mass x y z">
-        <inertial>
-            <mass value="${mass}" />
-            <inertia ixx="${1/12*mass*(y*y+z*z)}" ixy="0.0" ixz="0.0" iyy="${1/12*mass*(x*x+z*z)}" iyz="0.0" izz="${1/12*mass*(y*y+x*x)}" />
-        </inertial>
-    </xacro:macro>
+    <!-- Refer to Nav2's URDF tutorial -->
+    <!-- https://navigation.ros.org/setup_guides/urdf/setup_urdf.html -->
     <!-- define colors -->
-    <material name="blue">
-        <color rgba="0 0 0.8 1" />
-    </material>
     <material name="black">
         <color rgba="0 0 0 1" />
@@ -29,4 +13,67 @@
         <color rgba="0.3098 0.1765 0.4980 1" />
     </material>
+    <!-- Define robot constants -->
+    <!-- pi -->
+    <xacro:property name="PI" value="3.141592653589793" />
+    <!-- base properties -->
+    <xacro:property name="base_width" value="0.4" />
+    <xacro:property name="base_depth" value="0.2" />
+    <xacro:property name="base_height" value="0.1" />
+    <xacro:property name="base_mass" value="2.0" />
+    <!-- wheel properties -->
+    <xacro:property name="wheel_ygap" value="0.005" />
+    <xacro:property name="wheel_xoff" value="0.1" />
+    <xacro:property name="wheel_radius" value="0.1" />
+    <xacro:property name="wheel_width" value="0.05" />
+    <xacro:property name="wheel_mass" value="0.2" />
+    <!-- caster properties -->
+    <xacro:property name="caster_xoff" value="-0.15" />
+    <xacro:property name="caster_radius" value="0.05" />
+    <xacro:property name="caster_mass" value="0.3" />
+    <!-- Define intertial property macros  -->
+    <xacro:macro name="box_inertia" params="m w d h">
+        <inertial>
+            <origin xyz="0 0 0" rpy="${pi/2} 0 ${pi/2}" />
+            <mass value="${m}" />
+            <inertia ixx="${(m/12) * (h*h + d*d)}" ixy="0.0" ixz="0.0" iyy="${(m/12) * (w*w + h*h)}" iyz="0.0" izz="${(m/12) * (w*w + d*d)}" />
+        </inertial>
+    </xacro:macro>
+    <xacro:macro name="cylinder_inertia" params="m r h">
+        <inertial>
+            <origin xyz="0 0 0" rpy="${pi/2} 0 0" />
+            <mass value="${m}" />
+            <inertia ixx="${(m/12) * (3*r*r + h*h)}" ixy="0" ixz="0" iyy="${(m/12) * (3*r*r + h*h)}" iyz="0" izz="${(m/2) * (r*r)}" />
+        </inertial>
+    </xacro:macro>
+    <xacro:macro name="sphere_inertia" params="m r">
+        <inertial>
+            <mass value="${m}" />
+            <inertia ixx="${(2/5) * m * (r*r)}" ixy="0.0" ixz="0.0" iyy="${(2/5) * m * (r*r)}" iyz="0.0" izz="${(2/5) * m * (r*r)}" />
+        </inertial>
+    </xacro:macro>
+    <!-- Define wheel macros -->
+    <xacro:macro name="wheel" params="prefix y_reflect">
+        <joint name="${prefix}_joint" type="continuous">
+            <parent link="base_link" />
+            <child link="${prefix}_link" />
+            <origin xyz="${wheel_xoff} ${y_reflect*(base_depth/2+wheel_ygap+wheel_width/2)} 0" rpy="${PI/2} 0 0" />
+            <axis xyz="0 0 1" />
+        </joint>
+        <link name="${prefix}_link">
+            <visual>
+                <geometry>
+                    <cylinder radius="${wheel_radius}" length="${wheel_width}" />
+                </geometry>
+                <material name="black" />
+            </visual>
+            <collision>
+                <geometry>
+                    <cylinder radius="${wheel_radius}" length="${wheel_width}" />
+                </geometry>
+            </collision>
+            <xacro:cylinder_inertia m="${wheel_mass}" r="${wheel_radius}" h="${wheel_width}" />
+        </link>
+    </xacro:macro>
+    <!-- Robot Base -->
     <link name="base_link">
         <visual>
@@ -41,92 +88,39 @@
             </geometry>
         </collision>
+        <xacro:box_inertia m="${base_mass}" w="${base_width}" d="${base_depth}" h="${base_height}" />
     </link>
     <gazebo reference="base_link">
         <material>Gazebo/White</material>
     </gazebo>
-    <joint name="base_link-base_footprint" type="fixed">
-        <origin rpy="0 0 0" xyz="0 0 -0.15" />
+    <!-- Robot Footprint -->
+    <joint name="footprint_joint" type="fixed">
         <parent link="base_link" />
         <child link="base_footprint" />
+        <origin xyz="0.0 0.0 ${-(wheel_radius)}" rpy="0 0 0" />
     </joint>
-    <!-- Base footprint is on the ground under the robot -->
     <link name="base_footprint" />
-    <joint name="base_link-base_inertial" type="fixed">
-        <origin rpy="0 0 0" xyz="0 0 0" />
-        <parent link="base_link" />
-        <child link="base_inertial" />
-    </joint>
-    <!-- Inertial link stores the robot's inertial information -->
-    <link name="base_inertial">
-        <xacro:box_inertial mass="1" x="${base_width}" y="${base_depth}" z="${base_height}" />
-    </link>
-    <joint name="base_to_left_wheel" type="continuous">
-        <parent link="base_link" />
-        <child link="left_wheel" />
-        <origin rpy="${PI/2} 0 0" xyz="${x_offset} ${base_depth/2+wheel_gap+wheel_width/2} 0" />
-        <axis rpy="0 0 0" xyz="0 0 1" />
-    </joint>
-    <link name="left_wheel">
-        <visual>
-            <geometry>
-                <cylinder length="0.05" radius="0.1" />
-            </geometry>
-            <material name="black" />
-        </visual>
-        <collision>
-            <geometry>
-                <cylinder length="0.05" radius="0.1" />
-            </geometry>
-        </collision>
-        <inertial>
-            <mass value="0.1" />
-            <inertia ixx="0.1" ixy="0.0" ixz="0.0" iyy="0.1" iyz="0.0" izz="0.1" />
-        </inertial>
-    </link>
-    <gazebo reference="left_wheel">
+    <!-- Wheels -->
+    <xacro:wheel prefix="left_whleel" y_reflect="1" />
+    <gazebo reference="left_wheel_link">
         <mu1>1.0</mu1>
         <mu2>1.0</mu2>
         <material>Gazebo/Black</material>
     </gazebo>
-    <joint name="base_to_right_wheel" type="continuous">
-        <parent link="base_link" />
-        <child link="right_wheel" />
-        <origin rpy="${PI/2} 0 0" xyz="${x_offset} ${-(base_depth/2+wheel_gap+wheel_width/2)} 0" />
-        <!-- <origin rpy="1.5707963267948966 0 0" xyz="0.1 -0.13 0" /> -->
-        <axis rpy="0 0 0" xyz="0 0 1" />
-    </joint>
-    <link name="right_wheel">
-        <visual>
-            <geometry>
-                <cylinder length="0.05" radius="0.1" />
-            </geometry>
-            <material name="black" />
-        </visual>
-        <collision>
-            <geometry>
-                <cylinder length="0.05" radius="0.1" />
-            </geometry>
-        </collision>
-        <inertial>
-            <mass value="0.1" />
-            <inertia ixx="0.1" ixy="0.0" ixz="0.0" iyy="0.1" iyz="0.0" izz="0.1" />
-        </inertial>
-    </link>
-    <gazebo reference="right_wheel">
+    <xacro:wheel prefix="right_whleel" y_reflect="-1" />
+    <gazebo reference="right_wheel_link">
         <mu1>1.0</mu1>
         <mu2>1.0</mu2>
         <material>Gazebo/Black</material>
     </gazebo>
-    <joint name="base_to_caster" type="revolute">
+    <!-- Caster ball -->
+    <joint name="caster_joint" type="fixed">
         <parent link="base_link" />
         <child link="caster" />
-        <origin xyz="-0.15 0 -0.05" />
-        <limit lower="0" upper="0" effort="0" velocity="0" />
-        <axis rpy="0 0 0" xyz="0 0 1" />
+        <origin xyz="${caster_xoff} 0.0 ${-(base_height/2)}" rpy="0 0 0" />
     </joint>
     <link name="caster">
         <visual>
             <geometry>
-                <sphere radius="0.05" />
+                <sphere radius="${caster_radius}" />
             </geometry>
             <material name="purple" />
@@ -134,11 +128,8 @@
         <collision>
             <geometry>
-                <sphere radius="0.05" />
+                <sphere radius="${caster_radius}" />
             </geometry>
         </collision>
-        <inertial>
-            <mass value="0.2" />
-            <inertia ixx="0.1" ixy="0.0" ixz="0.0" iyy="0.1" iyz="0.0" izz="0.1" />
-        </inertial>
+        <xacro:sphere_inertia m="${caster_mass}" r="${caster_radius}" />
     </link>
     <gazebo reference="caster">
@@ -150,16 +141,20 @@
     <gazebo>
         <plugin name="differential_drive_controller" filename="libgazebo_ros_diff_drive.so">
-            <!-- <ros>
+            <ros>
                 <namespace>/bot</namespace>
-                <argument>cmd_vel:=cmd_demo</argument>
-                <argument>odom:=odom_demo</argument>
-            </ros> -->
+                <!-- <argument>cmd_vel:=cmd_demo</argument>
+                <argument>odom:=odom_demo</argument> -->
+            </ros>
+            <robot_base_frame>base_link</robot_base_frame>
             <update_rate>100</update_rate>
-            <left_joint>base_to_left_wheel</left_joint>
-            <right_joint>base_to_right_wheel</right_joint>
+            <left_joint>left_wheel_joint</left_joint>
+            <right_joint>right_wheel_joint</right_joint>
             <wheel_separation>0.26</wheel_separation>
             <wheel_diameter>0.2</wheel_diameter>
+            <publish_odom>true</publish_odom>
+            <publish_odom_tf>false</publish_odom_tf>
+            <publish_wheel_tf>true</publish_wheel_tf>
             <odometry_frame>odom</odometry_frame>
-            <max_wheel_torque>20</max_wheel_torque>
+            <max_wheel_torque>10</max_wheel_torque>
             <!-- Wheel acceleration, in rad/s^2, defaults to 0.0 rad/s^2 -->
             <max_acceleration>1.0</max_acceleration>

Commit message: update urdf colors

File: urdf/bot.urdf.xacro (robot description, xacro)
@@ -12,4 +12,13 @@
     <material name="purple">
         <color rgba="0.3098 0.1765 0.4980 1" />
+    </material>
+    <material name="orange">
+        <color rgba="1 0.6471 0 1" />
+    </material>
+    <material name="navy">
+        <color rgba="0 0 0.5 1" />
+    </material>
+    <material name="gray">
+        <color rgba="0.5 0.5 0.5 1" />
     </material>
     <!-- Define robot constants -->
@@ -65,5 +74,5 @@
                     <cylinder radius="${wheel_radius}" length="${wheel_width}" />
                 </geometry>
-                <material name="black" />
+                <material name="navy" />
             </visual>
             <collision>
@@ -81,5 +90,5 @@
                 <box size="${base_width} ${base_depth} ${base_height}" />
             </geometry>
-            <material name="white" />
+            <material name="orange" />
         </visual>
         <collision>
@@ -91,5 +100,5 @@
     </link>
     <gazebo reference="base_link">
-        <material>Gazebo/White</material>
+        <material>Gazebo/Wood</material>
     </gazebo>
     <!-- Robot Footprint -->
@@ -105,5 +114,5 @@
         <mu1>1.0</mu1>
         <mu2>1.0</mu2>
-        <material>Gazebo/Black</material>
+        <material>Gazebo/Blue</material>
     </gazebo>
     <xacro:wheel prefix="right_wheel" y_reflect="-1" />
@@ -111,5 +120,5 @@
         <mu1>1.0</mu1>
         <mu2>1.0</mu2>
-        <material>Gazebo/Black</material>
+        <material>Gazebo/Blue</material>
     </gazebo>
     <!-- Caster ball -->
@@ -124,5 +133,5 @@
                 <sphere radius="${caster_radius}" />
             </geometry>
-            <material name="purple" />
+            <material name="gray" />
         </visual>
         <collision>
@@ -136,5 +145,5 @@
         <mu1>0.0</mu1>
         <mu2>0.0</mu2>
-        <material>Gazebo/Purple</material>
+        <material>Gazebo/Gray</material>
     </gazebo>
     <!-- differential_drive_controller plugin -->

Commit message: add lidar

File: urdf/bot.urdf.xacro (robot description, xacro)
@@ -40,4 +40,9 @@
     <xacro:property name="caster_radius" value="0.05" />
     <xacro:property name="caster_mass" value="0.3" />
+    <!-- lidar properties -->
+    <xacro:property name="lidar_radius" value="0.035" />
+    <xacro:property name="lidar_height" value="0.02" />
+    <xacro:property name="lidar_zoff" value="0.03" />
+    <xacro:property name="lidar_mass" value="0.17" />
     <!-- Define intertial property macros  -->
     <xacro:macro name="box_inertia" params="m w d h">
@@ -147,4 +152,61 @@
         <material>Gazebo/Gray</material>
     </gazebo>
+    <!-- lidar -->
+    <joint name="lidar_joint" type="fixed">
+        <parent link="base_link" />
+        <child link="lidar_link" />
+        <origin xyz="0 0 ${(base_height+lidar_height)/2+lidar_zoff}" rpy="0 0 0" />
+    </joint>
+    <link name="lidar_link">
+        <visual>
+            <origin xyz="0 0 0" rpy="0 0 0" />
+            <geometry>
+                <cylinder radius="${lidar_radius}" length="${lidar_height}" />
+            </geometry>
+            <material name="black" />
+        </visual>
+        <collision>
+            <origin xyz="0 0 0" rpy="0 0 0" />
+            <geometry>
+                <cylinder radius="${lidar_radius}" length="${lidar_height}" />
+            </geometry>
+        </collision>
+        <xacro:cylinder_inertia m="${lidar_mass}" r="${lidar_radius}" h="${lidar_height}" />
+    </link>
+    <gazebo reference="lidar_link">
+        <material>Gazebo/Black</material>
+        <sensor name="lidar" type="ray">
+            <always_on>true</always_on>
+            <visualize>true</visualize>
+            <update_rate>5</update_rate>
+            <ray>
+                <scan>
+                    <horizontal>
+                        <samples>360</samples>
+                        <resolution>1.000000</resolution>
+                        <min_angle>0.000000</min_angle>
+                        <max_angle>6.280000</max_angle>
+                    </horizontal>
+                </scan>
+                <range>
+                    <min>0.120000</min>
+                    <max>6</max>
+                    <resolution>0.015000</resolution>
+                </range>
+                <noise>
+                    <type>gaussian</type>
+                    <mean>0.0</mean>
+                    <stddev>0.01</stddev>
+                </noise>
+            </ray>
+            <plugin name="scan" filename="libgazebo_ros_ray_sensor.so">
+                <ros>
+                    <remapping>~/out:=scan</remapping>
+                </ros>
+                <output_type>sensor_msgs/LaserScan</output_type>
+                <frame_name>lidar_link</frame_name>
+            </plugin>
+        </sensor>
+    </gazebo>
     <!-- differential_drive_controller plugin -->
     <gazebo>
