Commit message: add imu link

File: urdf/bot.urdf.xacro (robot description, xacro)
@@ -45,4 +45,9 @@
     <xacro:property name="lidar_zoff" value="0.03" />
     <xacro:property name="lidar_mass" value="0.17" />
+    <!-- imu properties -->
+    <xacro:property name="imu_width" value="0.02" />
+    <xacro:property name="imu_depth" value="0.015" />
+    <xacro:property name="imu_height" value="0.001" />
+    <xacro:property name="imu_mass" value="0.002" />
     <!-- Define intertial property macros  -->
     <xacro:macro name="box_inertia" params="m w d h">
@@ -102,5 +107,4 @@
             </geometry>
         </collision>
-        <xacro:box_inertia m="${base_mass}" w="${base_width}" d="${base_depth}" h="${base_height}" />
     </link>
     <gazebo reference="base_link">
@@ -114,4 +118,13 @@
     </joint>
     <link name="base_footprint" />
+    <!-- Base Inertial -->
+    <joint name="base_inertial_joint" type="fixed">
+        <parent link="base_link" />
+        <child link="base_inertial" />
+        <origin xyz="0 0 0" rpy="0 0 0" />
+    </joint>
+    <link name="base_inertial">
+        <xacro:box_inertia m="${base_mass}" w="${base_width}" d="${base_depth}" h="${base_height}" />
+    </link>
     <!-- Wheels -->
     <xacro:wheel prefix="left_wheel" y_reflect="1" />
@@ -209,4 +222,24 @@
         </sensor>
     </gazebo>
+    <!-- imu -->
+    <joint name="imu_joint" type="fixed">
+        <parent link="base_link"/>
+        <child link="imu_link"/>
+        <origin xyz="${base_width/4} 0 ${(base_height+imu_height)/2}"/>
+    </joint>
+    <link name="imu_link">
+        <visual>
+            <geometry>
+                <box size="${imu_width} ${imu_depth} ${imu_height}"/>
+            </geometry>
+            <material name="purple" />
+        </visual>
+        <collision>
+            <geometry>
+                <box size="${imu_width} ${imu_depth} ${imu_height}"/>
+            </geometry>
+        </collision>
+        <xacro:box_inertia m="${imu_mass}" w="${imu_width}" d="${imu_depth}" h="${imu_height}" />
+    </link>
     <!-- differential_drive_controller plugin -->
     <gazebo>

Commit message: lift lidar so that wheels not block

File: urdf/bot.urdf.xacro (robot description, xacro)
@@ -43,5 +43,5 @@
     <xacro:property name="lidar_radius" value="0.035" />
     <xacro:property name="lidar_height" value="0.02" />
-    <xacro:property name="lidar_zoff" value="0.03" />
+    <xacro:property name="lidar_zoff" value="0.05" />
     <xacro:property name="lidar_mass" value="0.17" />
     <!-- imu properties -->

Commit message: orient wheels joint frame with -pi wrt base origin

File: urdf/bot.urdf.xacro (robot description, xacro)
@@ -76,5 +76,5 @@
             <parent link="base_link" />
             <child link="${prefix}_link" />
-            <origin xyz="${wheel_xoff} ${y_reflect*(base_depth/2+wheel_ygap+wheel_width/2)} 0" rpy="${PI/2} 0 0" />
+            <origin xyz="${wheel_xoff} ${y_reflect*(base_depth/2+wheel_ygap+wheel_width/2)} 0" rpy="${-PI/2} 0 0" />
             <axis xyz="0 0 1" />
         </joint>

Commit message: add gazebo ros plugin for imu

File: urdf/bot.urdf.xacro (robot description, xacro)
@@ -242,4 +242,73 @@
         <xacro:box_inertia m="${imu_mass}" w="${imu_width}" d="${imu_depth}" h="${imu_height}" />
     </link>
+    <gazebo reference="imu_link">
+        <material>Gazebo/Purple</material>
+        <sensor name="imu_sensor" type="imu">
+            <plugin filename="libgazebo_ros_imu_sensor.so" name="imu_plugin">
+                <ros>
+                    <namespace>/bot</namespace>
+                    <remapping>~/out:=imu</remapping>
+                </ros>
+                <initial_orientation_as_reference>false</initial_orientation_as_reference>
+            </plugin>
+            <always_on>true</always_on>
+            <update_rate>100</update_rate>
+            <visualize>true</visualize>
+            <imu>
+                <angular_velocity>
+                    <x>
+                        <noise type="gaussian">
+                            <mean>0.0</mean>
+                            <stddev>2e-4</stddev>
+                            <bias_mean>0.0000075</bias_mean>
+                            <bias_stddev>0.0000008</bias_stddev>
+                        </noise>
+                    </x>
+                    <y>
+                        <noise type="gaussian">
+                            <mean>0.0</mean>
+                            <stddev>2e-4</stddev>
+                            <bias_mean>0.0000075</bias_mean>
+                            <bias_stddev>0.0000008</bias_stddev>
+                        </noise>
+                    </y>
+                    <z>
+                        <noise type="gaussian">
+                            <mean>0.0</mean>
+                            <stddev>2e-4</stddev>
+                            <bias_mean>0.0000075</bias_mean>
+                            <bias_stddev>0.0000008</bias_stddev>
+                        </noise>
+                    </z>
+                </angular_velocity>
+                <linear_acceleration>
+                    <x>
+                        <noise type="gaussian">
+                            <mean>0.0</mean>
+                            <stddev>1.7e-2</stddev>
+                            <bias_mean>0.1</bias_mean>
+                            <bias_stddev>0.001</bias_stddev>
+                        </noise>
+                    </x>
+                    <y>
+                        <noise type="gaussian">
+                            <mean>0.0</mean>
+                            <stddev>1.7e-2</stddev>
+                            <bias_mean>0.1</bias_mean>
+                            <bias_stddev>0.001</bias_stddev>
+                        </noise>
+                    </y>
+                    <z>
+                        <noise type="gaussian">
+                            <mean>0.0</mean>
+                            <stddev>1.7e-2</stddev>
+                            <bias_mean>0.1</bias_mean>
+                            <bias_stddev>0.001</bias_stddev>
+                        </noise>
+                    </z>
+                </linear_acceleration>
+            </imu>
+        </sensor>
+    </gazebo>
     <!-- differential_drive_controller plugin -->
     <gazebo>
